Commit message: set up real robot

File: aloha_scripts/urdf/S1.urdf (robot description, URDF)
Before this commit: robot converted_robot, 21 links, 20 joints
Joints:
- joint Joint_Arm_0: axis 0.0 0.7071067811865476 -0.7071067811865476 -> 0.0 -0.7071067811865476 0.7071067811865476; limit lower=-3.141593 upper=3.141593 effort=100 velocity=100 -> lower=-2.79253 upper=2.79253 effort=1 velocity=0.09
- joint Joint_Arm_1: limit lower=-2.094395 upper=0.785398 effort=100 velocity=100 -> lower=-2.35619 upper=1.13446 effort=1 velocity=0.09
- joint Joint_Arm_2: limit lower=-3.141593 upper=3.141593 effort=100 velocity=100 -> lower=-2.79253 upper=2.79253 effort=1 velocity=0.09
- joint Joint_Arm_3: axis 1.0 0.0 0.0 -> -1.0 0.0 0.0; limit lower=-1.48353 upper=1.6580630000000003 effort=100 velocity=100 -> lower=-2.47 upper=0.76 effort=1 velocity=0.09
- joint Joint_Arm_4: limit lower=-3.141593 upper=3.141593 effort=100 velocity=100 -> lower=-2.79253 upper=2.79253 effort=1 velocity=0.09
- joint Joint_Arm_5: axis 1.0 0.0 0.0 -> -1.0 0.0 0.0; limit lower=-0.872665 upper=0.872665 effort=100 velocity=100 -> lower=-1.01229 upper=0.82030 effort=1 velocity=0.09
- joint Joint_Arm_6: axis 0.0 -0.7071067811865476 -0.7071067811865476 -> 0.0 0.7071067811865476 0.7071067811865476; limit lower=-0.872665 upper=0.872665 effort=100 velocity=100 -> lower=-0.872665 upper=0.872665 effort=1 velocity=0.09
